File: TROCA-MCU-STM32G474.kicad_pcb (KiCad board)
At the start: 4 copper layers, 130.5 x 93.2 mm, 47 parts, among them SW1 HX-3X6X2.5-X SMD TACT SWITCH, SW2 HX-3X6X2.5-X SMD TACT SWITCH, U3 STM32G474VETx, U4 74HC4051, X2 X32258MOB4SI

Commit message: ajustes 0.1
Routing:
- net +3.3V: track 347.6 -> 0.00 mm, vias 2 -> 0
- net /G_EN: track 276.7 -> 0.00 mm, vias 6 -> 0
- net /TIM1_CH1: track 262.1 -> 0.00 mm, vias 9 -> 0
- net /MOTOR1_INA: track 258.1 -> 0.00 mm, vias 9 -> 0
- net /MOTOR1_INB: track 238.9 -> 0.00 mm, vias 9 -> 0
- net /G_SEL_0: track 224.4 -> 0.00 mm, vias 10 -> 0
- net /SenseM1: track 207.4 -> 0.00 mm, vias 2 -> 0
- net /G_SEL_1: track 205.2 -> 0.00 mm, vias 5 -> 0
- net /MOTOR5_ENCB: track 195.2 -> 0.00 mm, vias 2 -> 0
- net /MOTOR6_ENCB: track 193.9 -> 0.00 mm, vias 2 -> 0
- net /MOTOR6_ENCA: track 181.5 -> 0.00 mm, vias 2 -> 0
- net /MOTOR5_ENCA: track 171.0 -> 0.00 mm, vias 1 -> 0
- net /MOTOR7_ENCB: track 163.8 -> 0.00 mm, vias 2 -> 0
- net /MOTOR7_ENCA: track 149.6 -> 0.00 mm, vias 2 -> 0
- net /MOTOR1_ENCA: track 123.7 -> 0.00 mm, vias 2 -> 0
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